Commit message: naniga?

File: urdf/robot.urdf.xacro (robot description, xacro)
@@ -33,5 +33,5 @@
     <inertial>
       <origin xyz="0.1 0 0.075"/>
-      <mass value="0.5"/>
+      <mass value="5.0"/>
       <inertia ixx="0.0046875" ixy="0.0" ixz="0.0" iyy="0.0046875" iyz="0.0" izz="0.0075"/>
     </inertial>
@@ -56,5 +56,5 @@
     </collision>
     <inertial>
-      <mass value="0.1"/>
+      <mass value="1.0"/>
       <inertia ixx="0.00007583" ixy="0.0" ixz="0.0" iyy="0.00007583" iyz="0.0" izz="0.000125"/>
     </inertial>
@@ -79,5 +79,5 @@
     </collision>
     <inertial>
-      <mass value="0.1"/>
+      <mass value="1.0"/>
       <inertia ixx="0.00007583" ixy="0.0" ixz="0.0" iyy="0.00007583" iyz="0.0" izz="0.000125"/>
     </inertial>
@@ -101,5 +101,5 @@
     </collision>
     <inertial>
-      <mass value="0.1"/>
+      <mass value="0.5"/>
       <inertia ixx="0.0001" ixy="0.0" ixz="0.0" iyy="0.0001" iyz="0.0" izz="0.0001"/>
     </inertial>
@@ -155,5 +155,5 @@
     	</collision>
     	<inertial>
-      		<mass value="0.5"/>
+      		<mass value="5.0"/>
       		<inertia ixx="0.0001" ixy="0" ixz="0" iyy="0.0001" iyz="0" izz="0.0001"/>
 		</inertial>
